Commit message: update urdf model.

File: pass_the_butter_description/robots/pass_the_butter.urdf (robot description, URDF)
Before this commit: robot pass_the_butter, 4 links, 3 joints
Links:
- link base: geometry visual cylinder length=0.012 radius=0.002; visual cylinder length=0.012 radius=0.002
Joints:
- joint base_base_link: origin xyz=0.0 0.0 2.7 rpy=0.0 0.0 0.0 -> xyz=0.0 0.0 0.0 rpy=0.0 0.0 0.0
- joint base_wheel_left: origin xyz=-0.175 0.0 0.0 rpy=1.570796 0.0 1.570796 -> xyz=-0.16 0.0 0.0 rpy=1.570796 0.0 1.570796
- joint base_wheel_right: origin xyz=0.175 0.0 0.0 rpy=1.570796 0.0 1.570796 -> xyz=0.16 0.0 0.0 rpy=1.570796 0.0 1.570796
